File: atmega_copier.brd (EAGLE design)
At the start: 48.2 x 31.8 mm, 18 parts, among them CN1 MINI-USB, IC1 ATMEGA328P, Q1 8 MHz, SW1 SWITCH

Commit message: v1.0 completed
Parts:
- added R5: 1.5k, resistor:R0805
Connections:
- net N$22 renamed RXD
- net N$23 renamed TXD
- net +5V: now also R5.2
- net N$1: now also R5.1
Routing:
- net +5V: track 110.7 -> 131.0 mm, vias 0 -> 2
- net N$1: track 11.9 -> 13.3 mm
Changed lines of the file:
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@@
 <layer number="25" name="tNames" color="7" fill="1" visible="yes" active="yes"/>
 <layer number="26" name="bNames" color="7" fill="1" visible="no" active="yes"/>
-<layer number="27" name="tValues" color="7" fill="1" visible="no" active="yes"/>
+<layer number="27" name="tValues" color="7" fill="1" visible="yes" active="yes"/>
 <layer number="28" name="bValues" color="7" fill="1" visible="no" active="yes"/>
 <layer number="29" name="tStop" color="7" fill="1" visible="no" active="yes"/>
@@
 <element name="R4" library="resistor" package="R0805" value="10k" x="33.02" y="3.81"/>
 <element name="SW1" library="buttons" package="BT4.5X4.5" value="SWITCH" x="27.94" y="7.62" rot="R270"/>
+<element name="R5" library="resistor" package="R0805" value="1.5k" x="23.45" y="26.15"/>
 </elements>
 <signals>
@@
 <contactref element="SW1" pad="S"/>
 <contactref element="CN1" pad="VBUS"/>
-<wire x1="7.874" y1="21.92" x2="13.03" y2="21.92" width="0.6096" layer="1"/>
+<wire x1="12.7" y1="21.92" x2="7.874" y2="21.92" width="0.6096" layer="1"/>
+<wire x1="12.7" y1="21.92" x2="13.03" y2="21.92" width="0.6096" layer="1"/>
 <wire x1="13.03" y1="21.92" x2="13.97" y2="22.86" width="0.6096" layer="1"/>
 <wire x1="13.97" y1="22.86" x2="16.83" y2="22.86" width="0.6096" layer="1"/>
@@
 <wire x1="43.18" y1="29.21" x2="47.29" y2="25.4" width="1.27" layer="1"/>
 <wire x1="47.29" y1="25.4" x2="47.29" y2="19.15" width="1.27" layer="1"/>
+<contactref element="R5" pad="2"/>
+<wire x1="24.4" y1="26.15" x2="25.92" y2="26.15" width="0.6096" layer="1"/>
+<wire x1="25.92" y1="26.15" x2="26.67" y2="25.4" width="0.6096" layer="1"/>
+<via x="26.67" y="25.4" extent="1-16" drill="0.9" shape="octagon"/>
+<wire x1="26.67" y1="25.4" x2="19.05" y2="25.4" width="0.6096" layer="16"/>
+<wire x1="19.05" y1="25.4" x2="13.97" y2="20.32" width="0.6096" layer="16"/>
+<wire x1="13.97" y1="20.32" x2="12.7" y2="20.32" width="0.6096" layer="16"/>
+<via x="12.7" y="20.32" extent="1-16" drill="0.9" shape="octagon"/>
+<wire x1="12.7" y1="20.32" x2="12.7" y2="21.92" width="0.6096" layer="1"/>
 <wire x1="26.44" y1="4.04" x2="26.44" y2="11.12" width="0" layer="19" extent="1-1"/>
 </signal>
@@
 <wire x1="31.369" y1="16.0084" x2="31.369" y2="12.761" width="0.6096" layer="1"/>
 </signal>
-<signal name="N$22">
+<signal name="RXD">
 <contactref element="JP2" pad="1"/>
 <contactref element="IC1" pad="30"/>
@@
 <wire x1="29.21" y1="30.48" x2="29.21" y2="27.94" width="1.27" layer="1"/>
 </signal>
-<signal name="N$23">
+<signal name="TXD">
 <contactref element="IC1" pad="31"/>
 <contactref element="JP2" pad="2"/>
@@
 <wire x1="27.4574" y1="23.12" x2="23.87" y2="23.12" width="0.6096" layer="1"/>
 <wire x1="23.87" y1="23.12" x2="21.59" y2="25.4" width="0.6096" layer="1"/>
-<wire x1="21.59" y1="25.4" x2="21.59" y2="29.21" width="1.27" layer="1"/>
+<wire x1="21.59" y1="26.67" x2="21.59" y2="25.4" width="1.27" layer="1"/>
+<wire x1="21.59" y1="26.67" x2="21.59" y2="29.21" width="1.27" layer="1"/>
 <wire x1="21.59" y1="29.21" x2="21.59" y2="30.48" width="1.27" layer="1"/>
+<contactref element="R5" pad="1"/>
+<wire x1="22.5" y1="26.15" x2="21.59" y2="26.15" width="0.6096" layer="1"/>
+<wire x1="21.59" y1="26.15" x2="21.59" y2="26.67" width="0.6096" layer="1"/>
 </signal>
 <signal name="N$2">
