File: atmega_copier.sch (EAGLE design)
At the start: 18 parts, among them CN1 MINI-USB, IC1 ATMEGA328P, Q1 8 MHz, SW1 SWITCH

Commit message: v1.0 completed
Parts:
- added R5: 1.5k, resistor:R-EU_R0805
Connections:
- net N$22 renamed RXD
- net N$23 renamed TXD
- net +5V: now also R5.2
- net N$1: now also R5.1
Changed lines of the file:
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@@
 <part name="R4" library="resistor" deviceset="R-EU_" device="R0805" value="10k"/>
 <part name="CN1" library="adafruit" deviceset="USB" device="MINIB" value="MINI-USB"/>
+<part name="R5" library="resistor" deviceset="R-EU_" device="R0805" value="1.5k"/>
 </parts>
 <sheets>
@@
 <instance part="R4" gate="G$1" x="129.54" y="38.1" rot="R270"/>
 <instance part="CN1" gate="G$1" x="167.64" y="60.96" rot="R180"/>
+<instance part="R5" gate="G$1" x="96.52" y="76.2" rot="R90"/>
 </instances>
 <busses>
@@
 <wire x1="157.48" y1="55.88" x2="147.32" y2="55.88" width="0.1524" layer="91"/>
 <junction x="147.32" y="55.88"/>
+<pinref part="R5" gate="G$1" pin="2"/>
+<wire x1="96.52" y1="81.28" x2="96.52" y2="83.82" width="0.1524" layer="91"/>
+<wire x1="96.52" y1="83.82" x2="104.14" y2="83.82" width="0.1524" layer="91"/>
 </segment>
 </net>
@@
 </segment>
 </net>
-<net name="N$22" class="0">
+<net name="RXD" class="0">
 <segment>
 <pinref part="JP2" gate="G$1" pin="1"/>
@@
 </segment>
 </net>
-<net name="N$23" class="0">
+<net name="TXD" class="0">
 <segment>
 <pinref part="IC1" gate="IC" pin="PD1(TXD/PCINT17)"/>
@@
 <wire x1="114.3" y1="50.8" x2="114.3" y2="60.96" width="0.1524" layer="91"/>
 <pinref part="IC1" gate="IC" pin="PD3(INT1/OC2B/PCINT19)"/>
-<wire x1="114.3" y1="60.96" x2="83.82" y2="60.96" width="0.1524" layer="91"/>
-</segment>
-</net>
+<wire x1="114.3" y1="60.96" x2="96.52" y2="60.96" width="0.1524" layer="91"/>
+<pinref part="R5" gate="G$1" pin="1"/>
+<wire x1="96.52" y1="60.96" x2="83.82" y2="60.96" width="0.1524" layer="91"/>
+<wire x1="96.52" y1="71.12" x2="96.52" y2="60.96" width="0.1524" layer="91"/>
+<junction x="96.52" y="60.96"/>
+</segment>
+</net>
